Commit message: Ported collisions to stl since Gazebo doesn't seem to create proper collisions using urdf for some reason

File: limo_gazebo/urdf/apartment.urdf.xacro (robot description, xacro)
@@ -5,5 +5,5 @@
       <origin xyz="0 0 0" rpy="0 0 0"/>
       <mass value="1"/>
-      <inertia ixx="1" ixy="0" ixz="0" iyy="1" iyz="0" izz="1"/>
+      <inertia ixx="0.16667" ixy="0" ixz="0" iyy="0.16667" iyz="0" izz="0.16667"/>
     </inertial>
     <visual>
@@ -16,5 +16,5 @@
       <origin xyz="0 0 0" rpy="0 0 0"/>
       <geometry>
-        <mesh filename="package://limo_gazebo/meshes/Structure.dae"/>
+        <mesh filename="package://limo_gazebo/meshes/Structure.stl"/>
       </geometry>
     </collision>

File: limo_gazebo/urdf/decorations.urdf.xacro (robot description, xacro)
@@ -5,5 +5,5 @@
       <origin xyz="0 0 0" rpy="0 0 0"/>
       <mass value="1"/>
-      <inertia ixx="1" ixy="0" ixz="0" iyy="1" iyz="0" izz="1"/>
+      <inertia ixx="0.16667" ixy="0" ixz="0" iyy="0.16667" iyz="0" izz="0.16667"/>
     </inertial>
     <visual>
@@ -16,5 +16,5 @@
       <origin xyz="0 0 0" rpy="0 0 0"/>
       <geometry>
-        <mesh filename="package://limo_gazebo/meshes/Decoration.dae"/>
+        <mesh filename="package://limo_gazebo/meshes/Decoration.stl"/>
       </geometry>
     </collision>
